File: fast_diode_pcb/_autosave-fast_diode_pcb.sch (KiCad schematic (older format))
At the start: 6 parts, among them J1 USB_B_Micro, J2 Conn_Coaxial, U1 LM358

Commit message: update to pcb and 1-clickbom.csv
Parts:
- C1: value C -> 1pF
- R1: value R_Small -> 1M
Changed lines of the file:
@@
 P 4350 3850
 F 0 "R1" V 4154 3850 50  0000 C CNN
-F 1 "R_Small" V 4245 3850 50  0000 C CNN
+F 1 "1M" V 4245 3850 50  0000 C CNN
 F 2 "Resistor_THT:R_Axial_DIN0207_L6.3mm_D2.5mm_P10.16mm_Horizontal" H 4350 3850 50  0001 C CNN
 F 3 "~" H 4350 3850 50  0001 C CNN
@@
 P 4450 4150
 F 0 "C1" V 4198 4150 50  0000 C CNN
-F 1 "C" V 4289 4150 50  0000 C CNN
+F 1 "1pF" V 4289 4150 50  0000 C CNN
 F 2 "Capacitor_THT:C_Disc_D4.3mm_W1.9mm_P5.00mm" H 4488 4000 50  0001 C CNN
 F 3 "~" H 4450 4150 50  0001 C CNN
@@
 BNC+
 $Comp
-L power:GNDREF #PWR?
+L power:GNDREF #PWR04
 U 1 1 5E58FB32
 P 4050 2300
-F 0 "#PWR?" H 4050 2050 50  0001 C CNN
+F 0 "#PWR04" H 4050 2050 50  0001 C CNN
 F 1 "GNDREF" V 4055 2172 50  0000 R CNN
 F 2 "" H 4050 2300 50  0001 C CNN
