File: fast_diode_pcb/fast_diode_pcb.kicad_pcb (KiCad board)
At the start: 2 copper layers, 48.9 x 29.2 mm, 7 parts, among them J1 USB_B_Micro, J2 Conn_Coaxial, U1 LM358

Commit message: board updates
Parts:
- R1: value 1 MOhm -> 1M
Routing:
- net GNDREF: track 0.00 -> 1.22 mm
Changed lines of the file:
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@@
-(kicad_pcb (version 20171130) (host pcbnew "(5.1.5)-3")
+(kicad_pcb (version 20171130) (host pcbnew 5.1.5-52549c5~84~ubuntu18.04.1)
   (general
     (thickness 1.6)
     (drawings 12)
-    (tracks 26)
+    (tracks 28)
     (zones 0)
     (modules 7)
@@
       (effects (font (size 1 1) (thickness 0.15)))
     )
-    (fp_text value "1 MOhm" (at 5.08 0 90) (layer F.SilkS)
+    (fp_text value 1M (at 5.08 0 90) (layer F.SilkS)
       (effects (font (size 1 1) (thickness 0.15)))
     )
@@
   (segment (start 149.86 102.87) (end 146.05 102.87) (width 0.25) (layer F.Cu) (net 2))
   (segment (start 146.05 102.87) (end 138.43 110.49) (width 0.25) (layer F.Cu) (net 2))
+  (segment (start 110.595 111.875) (end 110.68 111.79) (width 0.25) (layer F.Cu) (net 3))
+  (segment (start 110.595 112.9775) (end 110.595 111.875) (width 0.25) (layer F.Cu) (net 3))
   (segment (start 121.285 113.29) (end 121.285 114.09) (width 0.25) (layer F.Cu) (net 4))
   (segment (start 110.68 109.19) (end 117.185 109.19) (width 0.25) (layer F.Cu) (net 4))

Commit message: update pcb and prepare for kitspace
Other:
- board text added: "1"
Changed lines of the file:
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@@
   (general
     (thickness 1.6)
-    (drawings 12)
+    (drawings 13)
     (tracks 28)
     (zones 0)
@@
       (drillshape 0)
       (scaleselection 1)
-      (outputdirectory ""))
+      (outputdirectory "gerbers/"))
   )
   (net 0 "")
@@
     )
   )
+  (gr_text 1 (at 121.412 104.902 270) (layer F.SilkS)
+    (effects (font (size 1.5 1.5) (thickness 0.3)))
+  )
   (gr_line (start 106.68 114.935) (end 106.68 114.3) (layer Edge.Cuts) (width 0.05))
   (gr_line (start 106.68 116.205) (end 106.68 114.935) (layer Edge.Cuts) (width 0.05))
@@
   (segment (start 149.86 102.87) (end 146.05 102.87) (width 0.25) (layer F.Cu) (net 2))
   (segment (start 146.05 102.87) (end 138.43 110.49) (width 0.25) (layer F.Cu) (net 2))
-  (segment (start 110.595 111.875) (end 110.68 111.79) (width 0.25) (layer F.Cu) (net 3))
-  (segment (start 110.595 112.9775) (end 110.595 111.875) (width 0.25) (layer F.Cu) (net 3))
+  (segment (start 110.68 112.8925) (end 110.595 112.9775) (width 0.25) (layer F.Cu) (net 3))
+  (segment (start 110.68 111.79) (end 110.68 112.8925) (width 0.25) (layer F.Cu) (net 3))
   (segment (start 121.285 113.29) (end 121.285 114.09) (width 0.25) (layer F.Cu) (net 4))
   (segment (start 110.68 109.19) (end 117.185 109.19) (width 0.25) (layer F.Cu) (net 4))
